File: hardware/lped/schematics/accelerometer.kicad_sch (KiCad schematic)
At the start: 4 parts, among them U2 FXLS8974CF

Commit message: feat(hardware)!: v2 of LPED PCB
* Changed MCU to nRF52833 (from nRF52810)
* Added second LED
* Used specialized filter instead of discrete components for ANT
* Removed unnecessary pull-down resistor from miso
* Removed DOCK_BTN
Parts:
- removed R5: 10k, Resistor_SMD:R_0402_1005Metric, symbol Device:R_Small
- renumbered C10 to C5, C11 to C7
Changed lines of the file:
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@@
-	)
-	(junction
-		(at 105.41 96.52)
-		(diameter 0)
-		(color 0 0 0 0)
 	)
 	(junction
@@
 	(wire
 		(pts
-			(xy 88.9 92.71) (xy 120.65 92.71)
+			(xy 106.68 92.71) (xy 120.65 92.71)
 		)
 		(stroke
@@
 	(wire
 		(pts
-			(xy 102.87 96.52) (xy 105.41 96.52)
-		)
-		(stroke
-			(width 0)
-			(type default)
-		)
-	)
-	(wire
-		(pts
 			(xy 120.65 71.12) (xy 133.35 71.12)
 		)
@@
 	(wire
 		(pts
-			(xy 105.41 96.52) (xy 105.41 99.06)
-		)
-		(stroke
-			(width 0)
-			(type default)
-		)
-	)
-	(wire
-		(pts
 			(xy 111.76 71.12) (xy 120.65 71.12)
 		)
@@
 	(wire
 		(pts
-			(xy 88.9 93.98) (xy 88.9 92.71)
-		)
-		(stroke
-			(width 0)
-			(type default)
-		)
-	)
-	(wire
-		(pts
-			(xy 105.41 96.52) (xy 120.65 96.52)
+			(xy 106.68 93.98) (xy 106.68 92.71)
+		)
+		(stroke
+			(width 0)
+			(type default)
+		)
+	)
+	(wire
+		(pts
+			(xy 119.38 96.52) (xy 120.65 96.52)
 		)
 		(stroke
@@
 	(wire
 		(pts
-			(xy 105.41 104.14) (xy 105.41 105.41)
-		)
-		(stroke
-			(width 0)
-			(type default)
-		)
-	)
-	(wire
-		(pts
 			(xy 133.35 111.76) (xy 133.35 113.03)
 		)
@@
 	)
 	(label "BT_MODE"
-		(at 102.87 92.71 180)
+		(at 119.38 92.71 180)
 		(effects
 			(font
@@
 	(hierarchical_label "MISO"
 		(shape output)
-		(at 102.87 96.52 180)
+		(at 119.38 96.52 180)
 		(effects
 			(font
@@
 			)
 			(justify left)
-		)
-	)
-	(symbol
-		(lib_id "Device:R_Small")
-		(at 105.41 101.6 180)
-		(unit 1)
-		(exclude_from_sim no)
-		(in_bom yes)
-		(on_board yes)
-		(dnp yes)
-		(fields_autoplaced yes)
-		(property "Reference" "R5"
-			(at 107.95 100.3299 0)
-			(effects
-				(font
-					(size 1.27 1.27)
-				)
-				(justify right)
-			)
-		)
-		(property "Value" "10k"
-			(at 107.95 102.8699 0)
-			(effects
-				(font
-					(size 1.27 1.27)
-				)
-				(justify right)
-			)
-		)
-		(property "Footprint" "Resistor_SMD:R_0402_1005Metric"
-			(at 105.41 101.6 0)
-			(effects
-				(font
-					(size 1.27 1.27)
-				)
-				(hide yes)
-			)
-		)
-		(property "Datasheet" "~"
-			(at 105.41 101.6 0)
-			(effects
-				(font
-					(size 1.27 1.27)
-				)
-				(hide yes)
-			)
-		)
-		(property "Description" "Resistor, small symbol"
-			(at 105.41 101.6 0)
-			(effects
-				(font
-					(size 1.27 1.27)
-				)
-				(hide yes)
-			)
-		)
-		(pin "1"
-		)
-		(pin "2"
-		)
-		(instances
-			(project "schematics"
-				(path "/479b96bc-6d23-47e9-846e-8263fbfa5ee1/c7f83528-b221-4855-af9e-ac3fb8666c19"
-					(reference "R5")
-					(unit 1)
-				)
-			)
 		)
 	)
@@
 		(dnp no)
 		(fields_autoplaced yes)
-		(property "Reference" "C11"
+		(property "Reference" "C7"
 			(at 123.19 73.6662 0)
 			(effects
@@
 		)
 		(instances
-			(project "schematics"
-				(path "/479b96bc-6d23-47e9-846e-8263fbfa5ee1/c7f83528-b221-4855-af9e-ac3fb8666c19"
-					(reference "C11")
-					(unit 1)
-				)
-			)
-		)
-	)
-	(symbol
-		(lib_id "power:Earth")
-		(at 105.41 105.41 0)
-		(unit 1)
-		(exclude_from_sim no)
-		(in_bom yes)
-		(on_board yes)
-		(dnp no)
-		(fields_autoplaced yes)
-		(property "Reference" "#PWR025"
-			(at 105.41 111.76 0)
-			(effects
-				(font
-					(size 1.27 1.27)
-				)
-				(hide yes)
-			)
-		)
-		(property "Value" "Earth"
-			(at 105.41 110.49 0)
-			(effects
-				(font
-					(size 1.27 1.27)
-				)
-				(hide yes)
-			)
-		)
-		(property "Footprint" ""
-			(at 105.41 105.41 0)
-			(effects
-				(font
-					(size 1.27 1.27)
-				)
-				(hide yes)
-			)
-		)
-		(property "Datasheet" "~"
-			(at 105.41 105.41 0)
-			(effects
-				(font
-					(size 1.27 1.27)
-				)
-				(hide yes)
-			)
-		)
-		(property "Description" "Power symbol creates a global label with name \"Earth\""
-			(at 105.41 105.41 0)
-			(effects
-				(font
-					(size 1.27 1.27)
-				)
-				(hide yes)
-			)
-		)
-		(pin "1"
-		)
-		(instances
-			(project "schematics"
-				(path "/479b96bc-6d23-47e9-846e-8263fbfa5ee1/c7f83528-b221-4855-af9e-ac3fb8666c19"
-					(reference "#PWR025")
+			(project "lped"
+				(path "/479b96bc-6d23-47e9-846e-8263fbfa5ee1/13a683db-0547-4126-8968-dbfeaa1350a9"
+					(reference "C7")
 					(unit 1)
 				)
@@
 		)
 		(instances
-			(project "schematics"
-				(path "/479b96bc-6d23-47e9-846e-8263fbfa5ee1/c7f83528-b221-4855-af9e-ac3fb8666c19"
+			(project "lped"
+				(path "/479b96bc-6d23-47e9-846e-8263fbfa5ee1/13a683db-0547-4126-8968-dbfeaa1350a9"
 					(reference "#PWR026")
 					(unit 1)
@@
 	(symbol
 		(lib_id "power:Earth")
-		(at 88.9 93.98 0)
+		(at 106.68 93.98 0)
 		(unit 1)
 		(exclude_from_sim no)
@@
 		(dnp no)
 		(fields_autoplaced yes)
-		(property "Reference" "#PWR024"
-			(at 88.9 100.33 0)
+		(property "Reference" "#PWR012"
+			(at 106.68 100.33 0)
 			(effects
 				(font
@@
 		)
 		(property "Value" "Earth"
-			(at 88.9 99.06 0)
+			(at 106.68 99.06 0)
 			(effects
 				(font
@@
 		)
 		(property "Footprint" ""
-			(at 88.9 93.98 0)
+			(at 106.68 93.98 0)
 			(effects
 				(font
@@
 		)
 		(property "Datasheet" "~"
-			(at 88.9 93.98 0)
+			(at 106.68 93.98 0)
 			(effects
 				(font
@@
 		)
 		(property "Description" "Power symbol creates a global label with name \"Earth\""
-			(at 88.9 93.98 0)
+			(at 106.68 93.98 0)
 			(effects
 				(font
@@
 		)
 		(instances
-			(project "schematics"
-				(path "/479b96bc-6d23-47e9-846e-8263fbfa5ee1/c7f83528-b221-4855-af9e-ac3fb8666c19"
-					(reference "#PWR024")
+			(project "lped"
+				(path "/479b96bc-6d23-47e9-846e-8263fbfa5ee1/13a683db-0547-4126-8968-dbfeaa1350a9"
+					(reference "#PWR012")
 					(unit 1)
 				)
@@
 		(dnp no)
 		(fields_autoplaced yes)
-		(property "Reference" "#PWR014"
+		(property "Reference" "#PWR024"
 			(at 111.76 86.36 0)
 			(effects
@@
 		)
 		(instances
-			(project "schematics"
-				(path "/479b96bc-6d23-47e9-846e-8263fbfa5ee1/c7f83528-b221-4855-af9e-ac3fb8666c19"
-					(reference "#PWR014")
+			(project "lped"
+				(path "/479b96bc-6d23-47e9-846e-8263fbfa5ee1/13a683db-0547-4126-8968-dbfeaa1350a9"
+					(reference "#PWR024")
 					(unit 1)
 				)
@@
 		)
 		(instances
-			(project "schematics"
-				(path "/479b96bc-6d23-47e9-846e-8263fbfa5ee1/c7f83528-b221-4855-af9e-ac3fb8666c19"
+			(project "lped"
+				(path "/479b96bc-6d23-47e9-846e-8263fbfa5ee1/13a683db-0547-4126-8968-dbfeaa1350a9"
 					(reference "#PWR023")
 					(unit 1)
@@
 		(dnp no)
 		(fields_autoplaced yes)
-		(property "Reference" "C10"
+		(property "Reference" "C5"
 			(at 114.3 73.6662 0)
 			(effects
@@
 		)
 		(instances
-			(project "schematics"
-				(path "/479b96bc-6d23-47e9-846e-8263fbfa5ee1/c7f83528-b221-4855-af9e-ac3fb8666c19"
-					(reference "C10")
+			(project "lped"
+				(path "/479b96bc-6d23-47e9-846e-8263fbfa5ee1/13a683db-0547-4126-8968-dbfeaa1350a9"
+					(reference "C5")
 					(unit 1)
 				)
@@
 		(dnp no)
 		(fields_autoplaced yes)
-		(property "Reference" "#PWR013"
+		(property "Reference" "#PWR025"
 			(at 133.35 73.66 0)
 			(effects
@@
 		)
 		(instances
-			(project "schematics"
-				(path "/479b96bc-6d23-47e9-846e-8263fbfa5ee1/c7f83528-b221-4855-af9e-ac3fb8666c19"
-					(reference "#PWR013")
+			(project "lped"
+				(path "/479b96bc-6d23-47e9-846e-8263fbfa5ee1/13a683db-0547-4126-8968-dbfeaa1350a9"
+					(reference "#PWR025")
 					(unit 1)
 				)
@@
 		)
 		(instances
-			(project ""
-				(path "/479b96bc-6d23-47e9-846e-8263fbfa5ee1/c7f83528-b221-4855-af9e-ac3fb8666c19"
+			(project "lped"
+				(path "/479b96bc-6d23-47e9-846e-8263fbfa5ee1/13a683db-0547-4126-8968-dbfeaa1350a9"
 					(reference "U2")
 					(unit 1)
