File: hardware/lped_dock/schematics/usb.kicad_sch (KiCad schematic)
At the start: 5 parts, among them J7 USB-C connector, U1 TPD4E02B04DQA

Commit message: feat(hardware): remove unused parts from dock pcb
* Removed LED from dock
* Removed button from dock
* Removed connection pins for LED and button
Connections:
- net USB_CC1 is gone; now on net CC1: J7.A5 (CC1), U1.1 (IO1)
- net USB_CC2 is gone; now on net CC2: J7.B5 (CC2), U1.2 (IO2)
- net USB_D+ is gone; now on net D+: U1.5 (IO4)
- net USB_D- is gone; now on net D-: U1.4 (IO3)
Changed lines of the file:
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@@
+	)
+	(junction
+		(at 181.61 88.9)
+		(diameter 0)
+		(color 0 0 0 0)
+	)
+	(junction
+		(at 181.61 83.82)
+		(diameter 0)
+		(color 0 0 0 0)
+	)
+	(junction
+		(at 181.61 96.52)
+		(diameter 0)
+		(color 0 0 0 0)
+	)
+	(junction
+		(at 181.61 91.44)
+		(diameter 0)
+		(color 0 0 0 0)
+	)
+	(junction
+		(at 181.61 99.06)
+		(diameter 0)
+		(color 0 0 0 0)
+	)
+	(junction
+		(at 181.61 101.6)
+		(diameter 0)
+		(color 0 0 0 0)
+	)
+	(junction
+		(at 181.61 86.36)
+		(diameter 0)
+		(color 0 0 0 0)
 	)
 	(junction
@@
 		(color 0 0 0 0)
 	)
+	(junction
+		(at 181.61 104.14)
+		(diameter 0)
+		(color 0 0 0 0)
+	)
 	(no_connect
 		(at 130.81 100.33)
@@
 	(wire
 		(pts
+			(xy 181.61 96.52) (xy 181.61 99.06)
+		)
+		(stroke
+			(width 0)
+			(type default)
+		)
+	)
+	(wire
+		(pts
 			(xy 179.07 83.82) (xy 181.61 83.82)
 		)
@@
 	(wire
 		(pts
+			(xy 181.61 101.6) (xy 181.61 104.14)
+		)
+		(stroke
+			(width 0)
+			(type default)
+		)
+	)
+	(wire
+		(pts
 			(xy 179.07 91.44) (xy 181.61 91.44)
 		)
@@
 	(wire
 		(pts
+			(xy 181.61 88.9) (xy 181.61 91.44)
+		)
+		(stroke
+			(width 0)
+			(type default)
+		)
+	)
+	(wire
+		(pts
 			(xy 132.08 85.09) (xy 130.81 85.09)
 		)
@@
 		)
 		(stroke
+			(width 0)
+			(type default)
+		)
+	)
+	(wire
+		(pts
+			(xy 181.61 83.82) (xy 181.61 86.36)
+		)
+		(stroke
