File: hardware/lped_dock/single_dock/schematics/lped_dock.kicad_pcb (KiCad board)
At the start: 2 copper layers, 32 x 18 mm, 29 parts, among them IC1 BQ24050DSQR, J1 V_{OUT}, J2 CONN, J3 GND, J7 USB-C connector, U1 TPD4E02B04DQA, U3 TLV62080DSGx

Commit message: fix(hardware): minor fixes before manufacturing
Changed footprint of USB protection diode
Changed footprint of Programmer fuse
Parts:
- R10: footprint Resistor_SMD:R_0603_1608Metric -> Resistor_SMD:R_1206_3216Metric
- moved R10 1.02 mm to (123.3, 110.7)
Routing:
- net Net-(BT1-+): track 9.31 -> 8.62 mm
- net Earth: vias 32 -> 31
Changed lines of the file:
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@@
 		)
 	)
-	(footprint "Resistor_SMD:R_0603_1608Metric"
+	(footprint "Resistor_SMD:R_1206_3216Metric"
 		(layer "F.Cu")
-		(at 122.7 109.9 90)
-		(descr "Resistor SMD 0603 (1608 Metric), square (rectangular) end terminal, IPC-7351 nominal, (Body size source: IPC-SM-782 page 72, https://www.pcb-3d.com/wordpress/wp-content/uploads/ipc-sm-782a_amendment_1_and_2.pdf), generated with kicad-footprint-generator")
+		(at 123.32 110.71 90)
+		(descr "Resistor SMD 1206 (3216 Metric), square (rectangular) end terminal, IPC-7351 nominal, (Body size source: IPC-SM-782 page 72, https://www.pcb-3d.com/wordpress/wp-content/uploads/ipc-sm-782a_amendment_1_and_2.pdf), generated with kicad-footprint-generator")
 		(tags "resistor")
 		(property "Reference" "R10"
-			(at 0 -1.43 90)
+			(at 0 -1.83 90)
 			(layer "F.SilkS")
 			(hide yes)
@@
 		)
 		(property "Value" "18R"
-			(at 0 1.43 90)
+			(at 0 1.83 90)
 			(layer "F.Fab")
 			(effects
@@
 		(attr smd)
 		(fp_line
-			(start -0.237258 -0.5225)
-			(end 0.237258 -0.5225)
+			(start -0.727064 -0.91)
+			(end 0.727064 -0.91)
 			(stroke
 				(width 0.12)
@@
 		)
 		(fp_line
-			(start -0.237258 0.5225)
-			(end 0.237258 0.5225)
+			(start -0.727064 0.91)
+			(end 0.727064 0.91)
 			(stroke
 				(width 0.12)
@@
 		)
 		(fp_line
-			(start 1.48 -0.73)
-			(end 1.48 0.73)
+			(start 2.28 -1.13)
+			(end 2.28 1.13)
 			(stroke
 				(width 0.05)
@@
 		)
 		(fp_line
-			(start -1.48 -0.73)
-			(end 1.48 -0.73)
+			(start -2.28 -1.13)
+			(end 2.28 -1.13)
 			(stroke
 				(width 0.05)
@@
 		)
 		(fp_line
-			(start 1.48 0.73)
-			(end -1.48 0.73)
+			(start 2.28 1.13)
+			(end -2.28 1.13)
 			(stroke
 				(width 0.05)
@@
 		)
 		(fp_line
-			(start -1.48 0.73)
-			(end -1.48 -0.73)
+			(start -2.28 1.13)
+			(end -2.28 -1.13)
 			(stroke
 				(width 0.05)
@@
 		)
 		(fp_line
-			(start 0.8 -0.4125)
-			(end 0.8 0.4125)
+			(start 1.6 -0.8)
+			(end 1.6 0.8)
 			(stroke
 				(width 0.1)
@@
 		)
 		(fp_line
-			(start -0.8 -0.4125)
-			(end 0.8 -0.4125)
+			(start -1.6 -0.8)
+			(end 1.6 -0.8)
 			(stroke
 				(width 0.1)
@@
 		)
 		(fp_line
-			(start 0.8 0.4125)
-			(end -0.8 0.4125)
+			(start 1.6 0.8)
+			(end -1.6 0.8)
 			(stroke
 				(width 0.1)
@@
 		)
 		(fp_line
-			(start -0.8 0.4125)
-			(end -0.8 -0.4125)
+			(start -1.6 0.8)
+			(end -1.6 -0.8)
 			(stroke
 				(width 0.1)
@@
 			(effects
 				(font
-					(size 0.4 0.4)
-					(thickness 0.06)
+					(size 0.8 0.8)
+					(thickness 0.12)
 				)
 			)
 		)
 		(pad "1" smd roundrect
-			(at -0.825 0 90)
-			(size 0.8 0.95)
+			(at -1.4625 0 90)
+			(size 1.125 1.75)
 			(layers "F.Cu" "F.Mask" "F.Paste")
-			(roundrect_rratio 0.25)
+			(roundrect_rratio 0.222222)
 			(net 17 "Net-(F1-Pad2)")
 			(pintype "passive")
 		)
 		(pad "2" smd roundrect
-			(at 0.825 0 90)
-			(size 0.8 0.95)
+			(at 1.4625 0 90)
+			(size 1.125 1.75)
 			(layers "F.Cu" "F.Mask" "F.Paste")
-			(roundrect_rratio 0.25)
+			(roundrect_rratio 0.222222)
 			(net 3 "Net-(BT1-+)")
 			(pintype "passive")
 		)
 		(embedded_fonts no)
-		(model "${KICAD9_3DMODEL_DIR}/Resistor_SMD.3dshapes/R_0603_1608Metric.step"
+		(model "${KICAD9_3DMODEL_DIR}/Resistor_SMD.3dshapes/R_1206_3216Metric.step"
 			(offset
 				(xyz 0 0 0)
@@
 	)
 	(via
-		(at 123.86 111.24)
-		(size 0.6)
-		(drill 0.3)
-		(layers "F.Cu" "B.Cu")
-		(free yes)
-		(net 2)
-	)
-	(via
 		(at 128.94 108.7)
 		(size 0.6)
@@
 	)
 	(segment
-		(start 126.525 110.3)
-		(end 125.3 109.075)
+		(start 126.49 110.3)
+		(end 125.44 109.25)
 		(width 0.8)
 		(layer "F.Cu")
@@
 	)
 	(segment
-		(start 122.7 109.075)
-		(end 125.3 109.075)
+		(start 125.3675 109.2475)
+		(end 123.32 109.2475)
+		(width 0.8)
+		(layer "F.Cu")
+		(net 3)
+	)
+	(segment
+		(start 125.37 109.25)
+		(end 125.3675 109.2475)
 		(width 0.8)
 		(layer "F.Cu")
@@
 	(segment
 		(start 131.5 110.3)
-		(end 126.525 110.3)
+		(end 126.49 110.3)
+		(width 0.8)
+		(layer "F.Cu")
+		(net 3)
+	)
+	(segment
+		(start 125.44 109.25)
+		(end 125.37 109.25)
 		(width 0.8)
 		(layer "F.Cu")
@@
 	)
 	(segment
-		(start 122.075 110.725)
-		(end 122.7 110.725)
+		(start 123.2525 112.24)
+		(end 123.32 112.1725)
+		(width 0.8)
+		(layer "F.Cu")
+		(net 17)
+	)
+	(segment
+		(start 120.7725 112.1725)
+		(end 120.7 112.1)
 		(width 0.8)
 		(layer "F.Cu")
@@
 	)
 	(segment
-		(start 120.7 112.1)
-		(end 122.075 110.725)
+		(start 123.32 112.1725)
+		(end 120.7725 112.1725)
 		(width 0.8)
 		(layer "F.Cu")
@@
 	)
 	(zone
-		(net 4)
-		(net_name "3V6")
+		(net 2)
+		(net_name "Earth")
+		(layer "F.Cu")
+		(hatch edge 0.5)
+		(connect_pads yes
+			(clearance 0.2)
+		)
+		(min_thickness 0.2)
+		(filled_areas_thickness no)
+		(fill yes
+			(thermal_gap 0.5)
+			(thermal_bridge_width 0.5)
+			(smoothing fillet)
+			(radius 0.2)
+		)
+		(polygon
+			(pts
+				(xy 101.5 115.7) (xy 101.5 96) (xy 135.7 96) (xy 135.7 115.7)
+			)
+		)
+	)
+	(zone
+		(net 1)
+		(net_name "Net-(U3-VOS)")
 		(layer "F.Cu")
 		(name "$teardrop_padvia$")
 		(hatch none 0.1)
-		(priority 30000)
+		(priority 30001)
 		(attr
 			(teardrop
@@
 		(polygon
 			(pts
-				(xy 128.46 103.282707) (xy 129.26 103.282707) (xy 129.742707 101.675581) (xy 128.86 101.499) (xy 127.977293 101.675581)
+				(xy 125.808838 105.043154) (xy 125.243154 105.608838) (xy 126.025 106.080154) (xy 126.638207 105.600707)
+				(xy 126.025 104.818341)
 			)
 		)
 	)
 	(zone
-		(net 2)
-		(net_name "Earth")
+		(net 14)
+		(net_name "/Battery Charger/V_{BUS}")
 		(layer "F.Cu")
 		(hatch edge 0.5)
+		(priority 5)
 		(connect_pads yes
 			(clearance 0.2)
 		)
-		(min_thickness 0.2)
+		(min_thickness 0.25)
 		(filled_areas_thickness no)
 		(fill yes
@@
 		(polygon
 			(pts
-				(xy 101.5 115.7) (xy 101.5 96) (xy 135.7 96) (xy 135.7 115.7)
+				(xy 109.4 104.31) (xy 110.6 104.31) (xy 110.75 104.16) (xy 110.75 101.67) (xy 106.9 101.67) (xy 106.9 99.19)
+				(xy 111.64 99.19) (xy 111.64 102.4) (xy 113.25 102.4) (xy 113.25 104.91) (xy 109.41 104.91) (xy 109.4 104.9)
 			)
 		)
 	)
 	(zone
-		(net 14)
-		(net_name "/Battery Charger/V_{BUS}")
+		(net 4)
+		(net_name "3V6")
 		(layer "F.Cu")
-		(hatch edge 0.5)
-		(priority 5)
+		(name "$teardrop_padvia$")
+		(hatch none 0.1)
+		(priority 30000)
+		(attr
+			(teardrop
+				(type padvia)
+			)
+		)
 		(connect_pads yes
-			(clearance 0.2)
+			(clearance 0)
 		)
-		(min_thickness 0.25)
+		(min_thickness 0.0254)
 		(filled_areas_thickness no)
 		(fill yes
 			(thermal_gap 0.5)
 			(thermal_bridge_width 0.5)
-			(smoothing fillet)
-			(radius 0.2)
+			(island_removal_mode 1)
+			(island_area_min 10)
 		)
 		(polygon
 			(pts
-				(xy 109.4 104.31) (xy 110.6 104.31) (xy 110.75 104.16) (xy 110.75 101.67) (xy 106.9 101.67) (xy 106.9 99.19)
-				(xy 111.64 99.19) (xy 111.64 102.4) (xy 113.25 102.4) (xy 113.25 104.91) (xy 109.41 104.91) (xy 109.4 104.9)
+				(xy 128.46 103.282707) (xy 129.26 103.282707) (xy 129.742707 101.675581) (xy 128.86 101.499) (xy 127.977293 101.675581)
 			)
 		)
@@
 	)
 	(zone
-		(net 1)
-		(net_name "Net-(U3-VOS)")
-		(layer "F.Cu")
-		(name "$teardrop_padvia$")
-		(hatch none 0.1)
-		(priority 30001)
-		(attr
-			(teardrop
-				(type padvia)
-			)
-		)
-		(connect_pads yes
-			(clearance 0)
-		)
-		(min_thickness 0.0254)
-		(filled_areas_thickness no)
-		(fill yes
-			(thermal_gap 0.5)
-			(thermal_bridge_width 0.5)
-			(island_removal_mode 1)
-			(island_area_min 10)
-		)
-		(polygon
-			(pts
-				(xy 125.808838 105.043154) (xy 125.243154 105.608838) (xy 126.025 106.080154) (xy 126.638207 105.600707)
-				(xy 126.025 104.818341)
-			)
-		)
-	)
-	(zone
 		(net 0)
 		(net_name "")
@@
 	)
 	(zone
-		(net 13)
-		(net_name "/Battery Charger/V_{SYS}")
-		(layer "B.Cu")
-		(name "$teardrop_padvia$")
-		(hatch none 0.1)
-		(priority 30001)
-		(attr
-			(teardrop
-				(type padvia)
-			)
-		)
-		(connect_pads yes
-			(clearance 0)
-		)
-		(min_thickness 0.0254)
-		(filled_areas_thickness no)
-		(fill yes
-			(thermal_gap 0.5)
-			(thermal_bridge_width 0.5)
-			(island_removal_mode 1)
-			(island_area_min 10)
-		)
-		(polygon
-			(pts
-				(xy 111.07 100.69) (xy 111.07 99.89) (xy 110.57 99.79) (xy 110.069 100.29) (xy 110.57 100.79)
-			)
-		)
-	)
-	(zone
 		(net 2)
 		(net_name "Earth")
@@
 		)
 	)
+	(zone
+		(net 13)
+		(net_name "/Battery Charger/V_{SYS}")
+		(layer "B.Cu")
+		(name "$teardrop_padvia$")
+		(hatch none 0.1)
+		(priority 30001)
+		(attr
+			(teardrop
+				(type padvia)
+			)
+		)
+		(connect_pads yes
+			(clearance 0)
+		)
+		(min_thickness 0.0254)
+		(filled_areas_thickness no)
+		(fill yes
+			(thermal_gap 0.5)
+			(thermal_bridge_width 0.5)
+			(island_removal_mode 1)
+			(island_area_min 10)
+		)
+		(polygon
+			(pts
+				(xy 111.07 100.69) (xy 111.07 99.89) (xy 110.57 99.79) (xy 110.069 100.29) (xy 110.57 100.79)
+			)
+		)
+	)
 	(group "ViaStitching Earth"
 		(members "002ad36b-b0e0-4442-8921-0a7daeb82517" "02b6ee99-1652-47c5-b780-b55c9ce5bea6"
 			"06f0396b-bd56-4089-a108-1fa6bf606893" "16b4fab5-e2d3-4e2f-b86e-ac517f1acdc6"
-			"2654b296-dce5-4483-8cc4-80a9c71ab3fe" "280f543e-b360-4264-84ac-cb0a4f305833"
-			"33f26413-cc36-4316-8ade-67f1859961dd" "34f5d92f-8cd4-4e30-901b-7778815b1a0e"
-			"39983474-180f-4393-a29b-b1383ec4dcf0" "49578070-cf9b-416f-af15-e96e3c5d064a"
-			"53428de8-0f49-48e0-a674-ddaa486f42d6" "6aea438b-96e7-4ed3-9567-a1130a6812c0"
+			"280f543e-b360-4264-84ac-cb0a4f305833" "33f26413-cc36-4316-8ade-67f1859961dd"
+			"34f5d92f-8cd4-4e30-901b-7778815b1a0e" "39983474-180f-4393-a29b-b1383ec4dcf0"
+			"49578070-cf9b-416f-af15-e96e3c5d064a" "53428de8-0f49-48e0-a674-ddaa486f42d6"
 			"7289b85e-69ac-4688-8764-db30e1cf64af" "74e9ac0d-3acc-40f5-a8dc-40de474915f1"
 			"79db3e5a-5539-4b4e-a26f-5835c3c6c403" "ac045dc6-e175-4364-b418-3ea8d38029cb"
 			"ac26ed3d-64b8-47dd-aa4a-4f4986ae3d7b" "b4645232-c8a6-48e7-89d6-dd886f0cf106"
-			"b7c8512d-700a-417e-810d-c8a9e6c2ffdf" "e56ef7de-58f4-4031-ae7e-6aad605a5ff7"
-			"f2f8194d-1eae-4ba1-8cdc-b077e0743008"
+			"b7c8512d-700a-417e-810d-c8a9e6c2ffdf" "f2f8194d-1eae-4ba1-8cdc-b077e0743008"
 		)
 	)
